File: Hardware/Breakout/Breakout.kicad_pcb (KiCad board)
At the start: 2 copper layers, 35.8 x 59.6 mm, 20 parts, among them J1 Conn_Coaxial, J2 9v_batt_in, U1 TDC7200PWR, U2 MAX7375AXR805+T, U3 BUF602ID, U4 MAX9011EUT+T

Commit message: More revisions and generated Gerbers
Parts:
- U3: footprint BUF602ID:D0008A_N -> SOIC127P600X175-8N:SOIC127P600X175-8N
- moved TP2 3.25 mm to (133.1, 107.3)
Routing:
- net Net-(J1-In): track 23.6 -> 41.2 mm
- net SDA: track 42.5 -> 46.0 mm
- net SCL: track 42.4 -> 45.9 mm
- net REFCLK: track 19.6 -> 16.2 mm
- net +3.3V: track 139.0 -> 140.7 mm
- net SPICLK: track 41.3 -> 42.0 mm
Other:
- board text added: "Board: Biarki Firmware: Hussain"
- board text added: "Cat Herding: Anthony Design: Nicolas & Reece"
- board text added: "UVIC ECE 449 Group #23"
