File: Hardware/Breakout/Breakout.kicad_sch (KiCad schematic)
At the start: 20 parts, among them J1 Conn_Coaxial, J2 9v_batt_in, U1 TDC7200PWR, U2 BUF602ID, U3 MAX9011EUT+T, U4 MAX7375AXR805+T

Commit message: More revisions and generated Gerbers
Parts:
- U2: footprint BUF602ID:D0008A_N -> SOIC127P600X175-8N:SOIC127P600X175-8N
Changed lines of the file:
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@@
       (effects (font (size 1.524 1.524)))
     )
-    (property "Footprint" "BUF602ID:D0008A_N" (at 154.94 125.73 0)
+    (property "Footprint" "SOIC127P600X175-8N:SOIC127P600X175-8N" (at 154.94 125.73 0)
       (effects (font (size 1.27 1.27) italic) hide)
     )
